Commit message: resolved git submodule issue in /src/bumperbot_cpp_examples; created URDF for bumperbot

File: src/bumperbot_description/urdf/bumperbot.urdf.xacro (robot description, xacro)
@@ -43,3 +43,29 @@
     <origin rpy="0 0 0" xyz="0 0.07 0"/>
   </joint>
+  <link name="caster_front_link">
+    <visual>
+      <origin rpy="0 0 0" xyz="0 0 0"/>
+      <geometry>
+        <mesh filename="package://bumperbot_description/meshes/caster_front_link.STL"/>
+      </geometry>
+    </visual>
+  </link>
+  <joint name="caster_front_joint" type="fixed">
+    <parent link="base_link"/>
+    <child link="caster_front_link"/>
+    <origin rpy="0 0 0" xyz="0.04755 0 -0.0275"/>
+  </joint>
+  <link name="caster_rear_link">
+    <visual>
+      <origin rpy="0 0 0" xyz="0 0 0"/>
+      <geometry>
+        <mesh filename="package://bumperbot_description/meshes/caster_rear_link.STL"/>
+      </geometry>
+    </visual>
+  </link>
+  <joint name="caster_rear_joint" type="fixed">
+    <parent link="base_link"/>
+    <child link="caster_rear_link"/>
+    <origin rpy="0 0 0" xyz="-0.04755 0 -0.0275"/>
+  </joint>
 </robot>
